File: SeaLegs/STM32.kicad_sch (KiCad schematic)
At the start: 3 parts

Commit message: updated requirements
Parts:
- removed C11, C13: 0.1uF, Capacitor_SMD:C_0402_1005Metric, symbol Device:C
- removed U1: ~, symbol LIS2DS12:LIS2DS12
- added J2: Conn_ARM_SWD_TagConnect_TC2030-NL, Connector:Tag-Connect_TC2030-IDC-NL_2x03_P1.27mm_Vertical, symbol Connector:Conn_ARM_SWD_TagConnect_TC2030-NL
- added U1: STM32WB55RGV6, VFQFN68-8x8mm, symbol STM32WB55RGV6:STM32WB55RGV6
Connections:
- no-connect marks 1 -> 0
Other:
- note removed: "I2C pullups are present at master"
- note removed: "INT pins are push-pull"
- note removed: "Place caps close to IC pin"
- note removed: "TODO: Figure out the bus situation here"
- note removed: "Tie CS to VDDIO For I2C operation"
